Commit message: testing with links 1

File: body.urdf (robot description, URDF)
Before this commit: robot robot, 1 links, 0 joints
Links:
- removed link Box
- added link Link0, mass 1; collision box size=1 1 1; visual box size=1 1 1
- added link Link1, mass 1; collision box size=1 1 1; visual box size=1 1 1
Joints:
- added joint Link0_Link1: type revolute, parent Link0, child Link1, origin xyz=0 0 1 rpy=0 0 0, axis 0 1 0, limit lower=-3.14159 upper=3.14159 effort=0.0 velocity=0.0

Commit message: many many links from slides

File: body.urdf (robot description, URDF)
Before this commit: robot robot, 3 links, 2 joints
Links:
- added link Link3, mass 1; collision box size=1 1 1; visual box size=1 1 1
- added link Link4, mass 1; collision box size=1 1 1; visual box size=1 1 1
- added link Link5, mass 1; collision box size=1 1 1; visual box size=1 1 1
- added link Link6, mass 1; collision box size=1 1 1; visual box size=1 1 1
Joints:
- added joint Link2_Link3: type revolute, parent Link2, child Link3, origin xyz=0 0.5 0.5 rpy=0 0 0, axis 0 1 0, limit lower=-3.14159 upper=3.14159 effort=0.0 velocity=0.0
- added joint Link3_Link4: type revolute, parent Link3, child Link4, origin xyz=0 1 0 rpy=0 0 0, axis 0 1 0, limit lower=-3.14159 upper=3.14159 effort=0.0 velocity=0.0
- added joint Link4_Link5: type revolute, parent Link4, child Link5, origin xyz=0 0.5 -0.5 rpy=0 0 0, axis 0 1 0, limit lower=-3.14159 upper=3.14159 effort=0.0 velocity=0.0
- added joint Link5_Link6: type revolute, parent Link5, child Link6, origin xyz=0 0 -0.5 rpy=0 0 0, axis 0 1 0, limit lower=-3.14159 upper=3.14159 effort=0.0 velocity=0.0

Commit message: working on joints assignment

File: body.urdf (robot description, URDF)
Before this commit: robot robot, 7 links, 6 joints
Links:
- removed link Link0
- removed link Link1
- removed link Link2
- removed link Link3
- removed link Link4
- removed link Link5
- removed link Link6
- added link FrontLeg, mass 1; collision box size=1 1 1; visual box size=1 1 1
- added link Torso, mass 1; collision box size=1 1 1; visual box size=1 1 1
Joints:
- removed joint Link0_Link1
- removed joint Link1_Link2
- removed joint Link2_Link3
- removed joint Link3_Link4
- removed joint Link4_Link5
- removed joint Link5_Link6
- added joint Torso_FrontLeg: type revolute, parent Torso, child FrontLeg, origin xyz=0.5 0 -0.5 rpy=0 0 0, axis 0 1 0, limit lower=-3.14159 upper=3.14159 effort=0.0 velocity=0.0

Commit message: finished work on joints

File: body.urdf (robot description, URDF)
Before this commit: robot robot, 2 links, 1 joints
Links:
- added link BackLeg, mass 1; collision box size=1 1 1; visual box size=1 1 1
Joints:
- added joint Torso_BackLeg: type revolute, parent Torso, child BackLeg, origin xyz=1 0 1 rpy=0 0 0, axis 0 1 0, limit lower=-3.14159 upper=3.14159 effort=0.0 velocity=0.0
- joint Torso_FrontLeg: origin xyz=0.5 0 -0.5 rpy=0 0 0 -> xyz=2 0 1 rpy=0 0 0
